File: workshop_drum1/workshop_drum1.sch (KiCad schematic (older format))
At the start: 3 parts

Commit message: test#2
Parts:
- J1: renamed from J?; footprint (none) -> zfoot:Jack_Instrument
- gave numbers to parts that had none: 2
Changed lines of the file:
@@
 LIBS:contrib
 LIBS:valves
+LIBS:workshop_drum1-cache
 EELAYER 26 0
 EELAYER END
@@
 $EndDescr
 $Comp
-L HEX_INV_TRI U?
+L HEX_INV_TRI U1
 U 1 1 5A32441C
 P 2650 2600
-F 0 "U?" H 2675 2933 60  0000 C CNN
+F 0 "U1" H 2675 2933 60  0000 C CNN
 F 1 "HEX_INV_TRI" H 2675 2854 25  0000 C CNN
 F 2 "" H 2600 3250 60  0001 C CNN
@@
 $EndComp
 $Comp
-L ADS8634 U?
+L ADS8634 U2
 U 1 1 5A324491
 P 6350 2300
-F 0 "U?" H 6275 3500 60  0000 C CNN
+F 0 "U2" H 6275 3500 60  0000 C CNN
 F 1 "ADS8634" H 6275 3394 60  0000 C CNN
 F 2 "" H 6550 2250 60  0001 C CNN
@@
 $EndComp
 $Comp
-L JACK-MONO J?
+L JACK-MONO J1
 U 1 1 5A3244E4
 P 4450 4650
-F 0 "J?" H 4656 5037 60  0000 C CNN
+F 0 "J1" H 4656 5037 60  0000 C CNN
 F 1 "JACK-MONO" H 4656 4931 60  0000 C CNN
-F 2 "" H 4450 4650 60  0000 C CNN
+F 2 "zfoot:Jack_Instrument" H 4450 4650 60  0000 C CNN
 F 3 "" H 4450 4650 60  0000 C CNN
 	1    4450 4650

Commit message: started project
Parts:
- removed J1: JACK-MONO, zfoot:Jack_Instrument, symbol JACK-MONO
- removed U1: HEX_INV_TRI, symbol HEX_INV_TRI
- removed U2: ADS8634, symbol ADS8634
- added U? (x2): LM358, 4ms-footprints:DIP_8pin_TL082_TH, symbol LM358
- added U? (x6): HEX_INV_TRI, 4ms-footprints:DIP-14_W7.62mm, symbol HEX_INV_TRI
Changed lines of the file:
@@
 $EndDescr
 $Comp
-L HEX_INV_TRI U1
-U 1 1 5A32441C
-P 2650 2600
-F 0 "U1" H 2675 2933 60  0000 C CNN
-F 1 "HEX_INV_TRI" H 2675 2854 25  0000 C CNN
-F 2 "" H 2600 3250 60  0001 C CNN
-F 3 "" H 2600 3250 60  0001 C CNN
-	1    2650 2600
+L LM358 U?
+U 1 1 5A324A57
+P 2050 2350
+F 0 "U?" H 2391 2396 50  0000 L CNN
+F 1 "LM358" H 2391 2305 50  0000 L CNN
+F 2 "4ms-footprints:DIP_8pin_TL082_TH" H 2050 2350 50  0001 C CNN
+F 3 "" H 2050 2350 50  0001 C CNN
+	1    2050 2350
 	1    0    0    -1
 $EndComp
 $Comp
-L ADS8634 U2
-U 1 1 5A324491
-P 6350 2300
-F 0 "U2" H 6275 3500 60  0000 C CNN
-F 1 "ADS8634" H 6275 3394 60  0000 C CNN
-F 2 "" H 6550 2250 60  0001 C CNN
-F 3 "" H 6550 2250 60  0001 C CNN
-	1    6350 2300
+L LM358 U?
+U 2 1 5A324B18
+P 4100 2700
+F 0 "U?" H 4441 2746 50  0000 L CNN
+F 1 "LM358" H 4441 2655 50  0000 L CNN
+F 2 "4ms-footprints:DIP_8pin_TL082_TH" H 4100 2700 50  0001 C CNN
+F 3 "" H 4100 2700 50  0001 C CNN
+	2    4100 2700
 	1    0    0    -1
 $EndComp
 $Comp
-L JACK-MONO J1
-U 1 1 5A3244E4
-P 4450 4650
-F 0 "J1" H 4656 5037 60  0000 C CNN
-F 1 "JACK-MONO" H 4656 4931 60  0000 C CNN
-F 2 "zfoot:Jack_Instrument" H 4450 4650 60  0000 C CNN
-F 3 "" H 4450 4650 60  0000 C CNN
-	1    4450 4650
+L HEX_INV_TRI U?
+U 1 1 5A324BD2
+P 5350 3400
+F 0 "U?" H 5375 3733 60  0000 C CNN
+F 1 "HEX_INV_TRI" H 5375 3654 25  0000 C CNN
+F 2 "4ms-footprints:DIP-14_W7.62mm" H 5300 4050 60  0001 C CNN
+F 3 "" H 5300 4050 60  0001 C CNN
+	1    5350 3400
 	1    0    0    -1
 $EndComp
+$Comp
+L HEX_INV_TRI U?
+U 2 1 5A324E3E
+P 2400 3600
+F 0 "U?" H 2425 3933 60  0000 C CNN
+F 1 "HEX_INV_TRI" H 2425 3854 25  0000 C CNN
+F 2 "4ms-footprints:DIP-14_W7.62mm" H 2350 4250 60  0001 C CNN
+F 3 "" H 2350 4250 60  0001 C CNN
+	2    2400 3600
+	1    0    0    -1
+$EndComp
+$Comp
+L HEX_INV_TRI U?
+U 3 1 5A3250CC
+P 5600 1150
+F 0 "U?" H 5625 1483 60  0000 C CNN
+F 1 "HEX_INV_TRI" H 5625 1404 25  0000 C CNN
+F 2 "4ms-footprints:DIP-14_W7.62mm" H 5550 1800 60  0001 C CNN
+F 3 "" H 5550 1800 60  0001 C CNN
+	3    5600 1150
+	1    0    0    -1
+$EndComp
+$Comp
+L HEX_INV_TRI U?
+U 4 1 5A3251AB
+P 6400 1100
+F 0 "U?" H 6425 1433 60  0000 C CNN
+F 1 "HEX_INV_TRI" H 6425 1354 25  0000 C CNN
+F 2 "4ms-footprints:DIP-14_W7.62mm" H 6350 1750 60  0001 C CNN
+F 3 "" H 6350 1750 60  0001 C CNN
+	4    6400 1100
+	1    0    0    -1
+$EndComp
+$Comp
+L HEX_INV_TRI U?
+U 5 1 5A325203
+P 7050 1150
+F 0 "U?" H 7075 1483 60  0000 C CNN
+F 1 "HEX_INV_TRI" H 7075 1404 25  0000 C CNN
+F 2 "4ms-footprints:DIP-14_W7.62mm" H 7000 1800 60  0001 C CNN
+F 3 "" H 7000 1800 60  0001 C CNN
+	5    7050 1150
+	1    0    0    -1
+$EndComp
+$Comp
+L HEX_INV_TRI U?
+U 6 1 5A325300
+P 7700 1150
+F 0 "U?" H 7725 1483 60  0000 C CNN
+F 1 "HEX_INV_TRI" H 7725 1404 25  0000 C CNN
+F 2 "4ms-footprints:DIP-14_W7.62mm" H 7650 1800 60  0001 C CNN
+F 3 "" H 7650 1800 60  0001 C CNN
+	6    7700 1150
+	1    0    0    -1
+$EndComp

Commit message: ready to build schematic
Parts:
- added BB10, BB11, BB12, BB5, BB6, BB7, BB8, BB9: BreadBoardStrip, zfoot:BreadBoardStrip, symbol BreadBoardStrip
- added GND1, PWR1: GNDStrip, zfoot:GNDStrip, symbol GNDStrip
- added J?: 9v_Battery_Clip, zfoot:Jack_DC, symbol 9v_Battery_Clip
- added unit 7 of U2
- gave numbers to parts that had none: 2
Connections:
- net at U2.12: now also BB12.1
- net at U2.13: now also BB10.1
- new net: BB5.1, U2.1
- new net: BB7.1, U2.2
- new net: BB6.1, U2.5
- new net: BB8.1, U2.6
- new net: BB9.1, U2.3
- new net: BB11.1, U2.4
- new net: GND1.1, U2.7
- new net: PWR1.1, U2.14
Other:
- moved on the sheet: U2F
Changed lines of the file:
@@
-EESchema Schematic File Version 2
+EESchema Schematic File Version 3
 LIBS:4ms-headers
 LIBS:4ms-ic
@@
 $EndDescr
 $Comp
-L LM358 U?
+L LM358 U1
 U 1 1 5A324A57
 P 2050 2350
-F 0 "U?" H 2391 2396 50  0000 L CNN
+F 0 "U1" H 2391 2396 50  0000 L CNN
 F 1 "LM358" H 2391 2305 50  0000 L CNN
 F 2 "4ms-footprints:DIP_8pin_TL082_TH" H 2050 2350 50  0001 C CNN
@@
 $EndComp
 $Comp
-L LM358 U?
+L LM358 U1
 U 2 1 5A324B18
 P 4100 2700
-F 0 "U?" H 4441 2746 50  0000 L CNN
+F 0 "U1" H 4441 2746 50  0000 L CNN
 F 1 "LM358" H 4441 2655 50  0000 L CNN
 F 2 "4ms-footprints:DIP_8pin_TL082_TH" H 4100 2700 50  0001 C CNN
@@
 $EndComp
 $Comp
-L HEX_INV_TRI U?
-U 1 1 5A324BD2
+L HEX_INV_TRI U2
+U 5 1 5A324BD2
 P 5350 3400
-F 0 "U?" H 5375 3733 60  0000 C CNN
+F 0 "U2" H 5375 3733 60  0000 C CNN
 F 1 "HEX_INV_TRI" H 5375 3654 25  0000 C CNN
 F 2 "4ms-footprints:DIP-14_W7.62mm" H 5300 4050 60  0001 C CNN
 F 3 "" H 5300 4050 60  0001 C CNN
-	1    5350 3400
-	1    0    0    -1
-$EndComp
-$Comp
-L HEX_INV_TRI U?
-U 2 1 5A324E3E
-P 2400 3600
-F 0 "U?" H 2425 3933 60  0000 C CNN
-F 1 "HEX_INV_TRI" H 2425 3854 25  0000 C CNN
-F 2 "4ms-footprints:DIP-14_W7.62mm" H 2350 4250 60  0001 C CNN
-F 3 "" H 2350 4250 60  0001 C CNN
-	2    2400 3600
-	1    0    0    -1
-$EndComp
-$Comp
-L HEX_INV_TRI U?
-U 3 1 5A3250CC
-P 5600 1150
-F 0 "U?" H 5625 1483 60  0000 C CNN
-F 1 "HEX_INV_TRI" H 5625 1404 25  0000 C CNN
-F 2 "4ms-footprints:DIP-14_W7.62mm" H 5550 1800 60  0001 C CNN
-F 3 "" H 5550 1800 60  0001 C CNN
-	3    5600 1150
-	1    0    0    -1
-$EndComp
-$Comp
-L HEX_INV_TRI U?
-U 4 1 5A3251AB
-P 6400 1100
-F 0 "U?" H 6425 1433 60  0000 C CNN
-F 1 "HEX_INV_TRI" H 6425 1354 25  0000 C CNN
-F 2 "4ms-footprints:DIP-14_W7.62mm" H 6350 1750 60  0001 C CNN
-F 3 "" H 6350 1750 60  0001 C CNN
-	4    6400 1100
-	1    0    0    -1
-$EndComp
-$Comp
-L HEX_INV_TRI U?
-U 5 1 5A325203
-P 7050 1150
-F 0 "U?" H 7075 1483 60  0000 C CNN
-F 1 "HEX_INV_TRI" H 7075 1404 25  0000 C CNN
-F 2 "4ms-footprints:DIP-14_W7.62mm" H 7000 1800 60  0001 C CNN
-F 3 "" H 7000 1800 60  0001 C CNN
-	5    7050 1150
-	1    0    0    -1
-$EndComp
-$Comp
-L HEX_INV_TRI U?
+	5    5350 3400
+	1    0    0    -1
+$EndComp
+$Comp
+L HEX_INV_TRI U2
+U 4 1 5A324E3E
+P 2450 3600
+F 0 "U2" H 2475 3933 60  0000 C CNN
+F 1 "HEX_INV_TRI" H 2475 3854 25  0000 C CNN
+F 2 "4ms-footprints:DIP-14_W7.62mm" H 2400 4250 60  0001 C CNN
+F 3 "" H 2400 4250 60  0001 C CNN
+	4    2450 3600
+	1    0    0    -1
+$EndComp
+$Comp
+L HEX_INV_TRI U2
+U 1 1 5A3250CC
+P 6350 950
+F 0 "U2" H 6375 1283 60  0000 C CNN
+F 1 "HEX_INV_TRI" H 6375 1204 25  0000 C CNN
+F 2 "4ms-footprints:DIP-14_W7.62mm" H 6300 1600 60  0001 C CNN
+F 3 "" H 6300 1600 60  0001 C CNN
+	1    6350 950
+	1    0    0    -1
+$EndComp
+$Comp
+L HEX_INV_TRI U2
+U 3 1 5A3251AB
+P 6350 1750
+F 0 "U2" H 6375 2083 60  0000 C CNN
+F 1 "HEX_INV_TRI" H 6375 2004 25  0000 C CNN
+F 2 "4ms-footprints:DIP-14_W7.62mm" H 6300 2400 60  0001 C CNN
+F 3 "" H 6300 2400 60  0001 C CNN
+	3    6350 1750
+	1    0    0    -1
+$EndComp
+$Comp
+L HEX_INV_TRI U2
+U 2 1 5A325203
+P 7650 950
+F 0 "U2" H 7675 1283 60  0000 C CNN
+F 1 "HEX_INV_TRI" H 7675 1204 25  0000 C CNN
+F 2 "4ms-footprints:DIP-14_W7.62mm" H 7600 1600 60  0001 C CNN
+F 3 "" H 7600 1600 60  0001 C CNN
+	2    7650 950
+	1    0    0    -1
+$EndComp
+$Comp
+L HEX_INV_TRI U2
 U 6 1 5A325300
-P 7700 1150
-F 0 "U?" H 7725 1483 60  0000 C CNN
-F 1 "HEX_INV_TRI" H 7725 1404 25  0000 C CNN
-F 2 "4ms-footprints:DIP-14_W7.62mm" H 7650 1800 60  0001 C CNN
-F 3 "" H 7650 1800 60  0001 C CNN
-	6    7700 1150
-	1    0    0    -1
-$EndComp
+P 7700 1650
+F 0 "U2" H 7725 1983 60  0000 C CNN
+F 1 "HEX_INV_TRI" H 7725 1904 25  0000 C CNN
+F 2 "4ms-footprints:DIP-14_W7.62mm" H 7650 2300 60  0001 C CNN
+F 3 "" H 7650 2300 60  0001 C CNN
+	6    7700 1650
+	1    0    0    -1
+$EndComp
+$Comp
+L BreadBoardStrip BB5
+U 1 1 5A32DFC0
+P 6150 950
+F 0 "BB5" H 6209 829 60  0000 C CNN
+F 1 "BreadBoardStrip" H 6209 895 10  0000 C CNN
+F 2 "zfoot:BreadBoardStrip" H 6020 930 60  0001 C CNN
+F 3 "" H 6150 950 60  0001 C CNN
+	1    6150 950
+	-1   0    0    1
+$EndComp
+$Comp
+L BreadBoardStrip BB7
+U 1 1 5A32E0DC
+P 6600 950
+F 0 "BB7" H 6759 987 60  0000 L CNN
+F 1 "BreadBoardStrip" H 6759 921 10  0000 L CNN
+F 2 "zfoot:BreadBoardStrip" H 6470 930 60  0001 C CNN
+F 3 "" H 6600 950 60  0001 C CNN
+	1    6600 950
+	1    0    0    -1
+$EndComp
+$Comp
+L BreadBoardStrip BB8
+U 1 1 5A32E1BF
+P 6600 1750
+F 0 "BB8" H 6759 1787 60  0000 L CNN
+F 1 "BreadBoardStrip" H 6759 1721 10  0000 L CNN
+F 2 "zfoot:BreadBoardStrip" H 6470 1730 60  0001 C CNN
+F 3 "" H 6600 1750 60  0001 C CNN
+	1    6600 1750
+	1    0    0    -1
+$EndComp
+$Comp
+L BreadBoardStrip BB11
+U 1 1 5A32E1FA
+P 7900 950
+F 0 "BB11" H 8059 987 60  0000 L CNN
+F 1 "BreadBoardStrip" H 8059 921 10  0000 L CNN
+F 2 "zfoot:BreadBoardStrip" H 7770 930 60  0001 C CNN
+F 3 "" H 7900 950 60  0001 C CNN
+	1    7900 950
+	1    0    0    -1
+$EndComp
+$Comp
+L BreadBoardStrip BB12
+U 1 1 5A32E2E4
+P 7950 1650
+F 0 "BB12" H 8109 1687 60  0000 L CNN
+F 1 "BreadBoardStrip" H 8109 1621 10  0000 L CNN
+F 2 "zfoot:BreadBoardStrip" H 7820 1630 60  0001 C CNN
+F 3 "" H 7950 1650 60  0001 C CNN
+	1    7950 1650
+	1    0    0    -1
+$EndComp
+$Comp
+L BreadBoardStrip BB9
+U 1 1 5A32E61E
+P 7450 950
+F 0 "BB9" H 7509 829 60  0000 C CNN
+F 1 "BreadBoardStrip" H 7509 895 10  0000 C CNN
+F 2 "zfoot:BreadBoardStrip" H 7320 930 60  0001 C CNN
+F 3 "" H 7450 950 60  0001 C CNN
+	1    7450 950
+	-1   0    0    1
+$EndComp
+$Comp
+L BreadBoardStrip BB10
+U 1 1 5A32E668
+P 7500 1650
+F 0 "BB10" H 7559 1529 60  0000 C CNN
+F 1 "BreadBoardStrip" H 7559 1595 10  0000 C CNN
+F 2 "zfoot:BreadBoardStrip" H 7370 1630 60  0001 C CNN
+F 3 "" H 7500 1650 60  0001 C CNN
+	1    7500 1650
+	-1   0    0    1
+$EndComp
+$Comp
+L BreadBoardStrip BB6
+U 1 1 5A32E6B1
+P 6150 1750
+F 0 "BB6" H 6209 1629 60  0000 C CNN
+F 1 "BreadBoardStrip" H 6209 1695 10  0000 C CNN
+F 2 "zfoot:BreadBoardStrip" H 6020 1730 60  0001 C CNN
+F 3 "" H 6150 1750 60  0001 C CNN
+	1    6150 1750
+	-1   0    0    1
+$EndComp
+$Comp
+L GNDStrip GND1
+U 1 1 5A32F5DA
+P 5400 3700
+F 0 "GND1" H 5559 3737 15  0000 L CNN
+F 1 "GNDStrip" H 5559 3706 10  0000 L CNN
+F 2 "zfoot:GNDStrip" H 5270 3680 60  0001 C CNN
+F 3 "" H 5400 3700 60  0001 C CNN
+	1    5400 3700
+	1    0    0    -1
+$EndComp
+$Comp
+L HEX_INV_TRI U2
+U 7 1 5A3302AD
+P 5350 3400
+F 0 "U2" H 5375 3733 60  0000 C CNN
+F 1 "HEX_INV_TRI" H 5375 3654 25  0000 C CNN
+F 2 "4ms-footprints:DIP-14_W7.62mm" H 5300 4050 60  0001 C CNN
+F 3 "" H 5300 4050 60  0001 C CNN
+	7    5350 3400
+	1    0    0    -1
+$EndComp
+$Comp
+L GNDStrip PWR1
+U 1 1 5A330F13
+P 5400 3100
+F 0 "PWR1" H 5559 3137 15  0000 L CNN
+F 1 "GNDStrip" H 5559 3106 10  0000 L CNN
+F 2 "zfoot:GNDStrip" H 5270 3080 60  0001 C CNN
+F 3 "" H 5400 3100 60  0001 C CNN
+	1    5400 3100
+	1    0    0    -1
+$EndComp
+Wire Wire Line
+	5350 3150 5350 3100
+Wire Wire Line
+	5350 3100 5400 3100
+Wire Wire Line
+	5350 3650 5350 3700
+Wire Wire Line
+	5350 3700 5400 3700
+$Comp
+L 9v_Battery_Clip J?
+U 1 1 5A331B93
+P 2150 6400
+F 0 "J?" H 2181 6837 60  0000 C CNN
+F 1 "9v_Battery_Clip" H 2181 6731 60  0000 C CNN
+F 2 "zfoot:Jack_DC" H 2150 6400 60  0001 C CNN
+F 3 "" H 2150 6400 60  0001 C CNN
+	1    2150 6400
+	1    0    0    -1
+$EndComp

Commit message: schematic laid out - started PCB
Parts:
- added BB1: BreadBoardStrip, zfoot:BreadBoardStrip, symbol BreadBoardStrip
- added Button_ON1, PWR2, Switch_On1: SPST_small, zfoot:SPST_Wired, symbol SPST_small
- added C1: 100uF, 4ms-footprints:Cap_Electrolytic_TH, symbol CAP-ELEC-TH
- added C2, C4: 1uF, 4ms-footprints:Cap_Electrolytic_TH, symbol CAP-ELEC-TH
- added C3: 10uF, 4ms-footprints:Cap_Electrolytic_TH, symbol CAP-ELEC-TH
- added C5: 220nF, 4ms-footprints:Cap_Ceramic_TH, symbol CAP_TH
- added D1: 4002, 4ms-footprints:Diode_BAT-85S_TH, symbol DIODE_TH
- added D2: 4148, 4ms-footprints:Diode_BAT-85S_TH, symbol DIODE_TH
- added DECAY1: A500k-A1M, zfoot:Pot_Wired, symbol POT
- added J2: Trigger_Input, zfoot:Jack_Instrument, symbol JACK-TIP_GND
- added J3: Output, zfoot:Jack_Instrument, symbol JACK-TIP_GND
- added ON/OFF_LED1, Trig_LED1: LED-C1-A2, LED-C1-A2-3MM-VERT, symbol LED-C1-A2
- added Osc_Select1: SPDT_small, zfoot:SPDT_Wired, symbol SPDT_small
- added PITCH1: B50k, zfoot:Pot_Wired, symbol POT
- added R1, R2, R3, R7: 1k, 4ms-footprints:Resistor_TH_300, symbol RTH
- added R4: 1M, 4ms-footprints:Resistor_TH_300, symbol RTH
- added R5: 100k, 4ms-footprints:Resistor_TH_300, symbol RTH
- added R6, R8: 470, 4ms-footprints:Resistor_TH_300, symbol RTH
- added SENSE/STARVE1: A50k, zfoot:Pot_Wired, symbol POT
- added U3: 78L05, 4ms-footprints:TO-92_Molded_Narrow, symbol 78L05
- PWR1: value GNDStrip -> PWRStrip
- U2: value HEX_INV_TRI -> 7414
- gave numbers to parts that had none: 1
Connections:
- net at U1.1: now also D2.2 (A), R4.1
- net at U1.2 (-): now also R2.1, R4.2
- net at U1.3 (+): now also SENSE/STARVE1.2 (Center)
- net GND: now reaches U1.4 (V-)
- net GND: now also J1.2 (GND), U1.4 (V-), U2.9, C1.2 (-), C2.2 (-), C3.2 (-), C4.2 (-), DECAY1.1 (Left), J2.2 (GND), J3.2 (GND), R2.2, R3.2, R8.1, SENSE/STARVE1.3 (Right), U3.2 (GND)
- net +5V: now reaches U1.8 (V+)
- net +5V: now also U1.8 (V+), Button_ON1.2, C3.1 (+), Switch_On1.2, U3.3 (VO)
- net at U1.5 (+): now also C2.1 (+), D2.1 (K), R5.2
- net at U1.6 (-): now also PWR1.1, U1.7, U2.14
- net at U2.10: now also Osc_Select1.1, PITCH1.3 (Right)
- net at U2.11: now also C4.1 (+), R6.1
- net at U2.8: now also Trig_LED1.2 (A)
- net at J1.1 (9v): now also PWR2.2
- new net: C5.1, R7.1
- new net: J3.1 (V), R7.2
- new net: R8.2, Trig_LED1.1 (C)
- new net: C1.1 (+), D1.1 (K), U3.1 (VI)
- new net: D1.2 (A), ON/OFF_LED1.2 (A), PWR2.1
- new net: ON/OFF_LED1.1 (C), R3.1
- new net: C5.2, Osc_Select1.2
- new net: BB1.1, Osc_Select1.3
- new net: Button_ON1.1, R1.2, Switch_On1.1
- new net: J2.1 (V), R1.1, SENSE/STARVE1.1 (Left)
- new net: DECAY1.2 (Center), DECAY1.3 (Right), R5.1
- new net: PITCH1.1 (Left), PITCH1.2 (Center), R6.2
Other:
- note added: "design by ZD"
- moved on the sheet: BB10, BB11, BB12, BB5, BB6, BB7, BB8, BB9, GND1, J1, PWR1, U1A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

Commit message: finished first look of schematic
Parts:
- ON/OFF_LED1, Trig_LED1: footprint LED-C1-A2-3MM-VERT -> zfoot:LED_wired
Connections:
- net at D2.2 (A), R4.1: now also U1.7; no longer U1.1
- net at R2.1, R4.2: now also U1.6 (-); no longer U1.2 (-)
- net at SENSE/STARVE1.2 (Center): now also U1.5 (+); no longer U1.3 (+)
- net at C2.1 (+), D2.1 (K), R5.2: now also U1.3 (+); no longer U1.5 (+)
- net at PWR1.1, U2.14: now also U1.1, U1.2 (-); no longer U1.6 (-), U1.7
Changed lines of the file:
@@
 $Comp
 L LM358 U1
-U 1 1 5A324A57
+U 2 1 5A324A57
 P 2450 1650
 F 0 "U1" H 2400 1900 50  0000 L CNN
@@
 F 2 "4ms-footprints:DIP_8pin_TL082_TH" H 2450 1650 50  0001 C CNN
 F 3 "" H 2450 1650 50  0001 C CNN
-	1    2450 1650
+	2    2450 1650
 	1    0    0    -1
 $EndComp
 $Comp
 L LM358 U1
-U 2 1 5A324B18
+U 1 1 5A324B18
 P 4200 1650
 F 0 "U1" H 4541 1696 50  0000 L CNN
@@
 F 2 "4ms-footprints:DIP_8pin_TL082_TH" H 4200 1650 50  0001 C CNN
 F 3 "" H 4200 1650 50  0001 C CNN
-	2    4200 1650
+	1    4200 1650
 	1    0    0    -1
 $EndComp
@@
 F 0 "ON/OFF_LED1" H 2300 3496 45  0000 C CNN
 F 1 "LED-C1-A2" H 2300 3580 45  0000 C CNN
-F 2 "LED-C1-A2-3MM-VERT" H 2280 3850 20  0001 C CNN
+F 2 "zfoot:LED_wired" H 2280 3850 20  0001 C CNN
 F 3 "" H 2250 3700 60  0001 C CNN
 	1    2250 3700
@@
 F 0 "Trig_LED1" H 6650 2596 45  0000 C CNN
 F 1 "LED-C1-A2" H 6650 2680 45  0000 C CNN
-F 2 "LED-C1-A2-3MM-VERT" H 6630 2950 20  0001 C CNN
+F 2 "zfoot:LED_wired" H 6630 2950 20  0001 C CNN
 F 3 "" H 6600 2800 60  0001 C CNN
 	1    6600 2800

Commit message: CRUISIN'
Parts:
- removed BB10, BB12: BreadBoardStrip, zfoot:BreadBoardStrip, symbol BreadBoardStrip
- renumbered BB5 to IN1, BB9 to IN2, BB6 to IN3, BB7 to OUT1, BB11 to OUT2, BB8 to OUT3, BB1 to OscSwitchStrip1
Connections:
- net at SENSE/STARVE1.2 (Center): now also U1.3 (+); no longer U1.5 (+)
- net at R2.1, R4.2: now also U1.2 (-); no longer U1.6 (-)
- net at D2.2 (A), R4.1: now also U1.1; no longer U1.7
- net at PWR1.1, U2.14: now also U1.6 (-), U1.7; no longer U1.1, U1.2 (-)
- net at C2.1 (+), D2.1 (K), R5.2: now also U1.5 (+); no longer U1.3 (+)
- no-connect marks 0 -> 2
Changed lines of the file:
@@
 $Comp
 L LM358 U1
-U 2 1 5A324A57
+U 1 1 5A324A57
 P 2450 1650
 F 0 "U1" H 2400 1900 50  0000 L CNN
@@
 F 2 "4ms-footprints:DIP_8pin_TL082_TH" H 2450 1650 50  0001 C CNN
 F 3 "" H 2450 1650 50  0001 C CNN
-	2    2450 1650
+	1    2450 1650
 	1    0    0    -1
 $EndComp
 $Comp
 L LM358 U1
-U 1 1 5A324B18
+U 2 1 5A324B18
 P 4200 1650
 F 0 "U1" H 4541 1696 50  0000 L CNN
@@
 F 2 "4ms-footprints:DIP_8pin_TL082_TH" H 4200 1650 50  0001 C CNN
 F 3 "" H 4200 1650 50  0001 C CNN
-	1    4200 1650
+	2    4200 1650
 	1    0    0    -1
 $EndComp
@@
 $EndComp
 $Comp
-L BreadBoardStrip BB5
+L BreadBoardStrip IN1
 U 1 1 5A32DFC0
 P 3300 900
-F 0 "BB5" H 3359 779 60  0000 C CNN
+F 0 "IN1" H 3359 779 60  0000 C CNN
 F 1 "BreadBoardStrip" H 3359 845 10  0000 C CNN
 F 2 "zfoot:BreadBoardStrip" H 3170 880 60  0001 C CNN
@@
 $EndComp
 $Comp
-L BreadBoardStrip BB7
+L BreadBoardStrip OUT1
 U 1 1 5A32E0DC
 P 3750 900
-F 0 "BB7" H 3909 937 60  0000 L CNN
+F 0 "OUT1" H 3909 937 60  0000 L CNN
 F 1 "BreadBoardStrip" H 3909 871 10  0000 L CNN
 F 2 "zfoot:BreadBoardStrip" H 3620 880 60  0001 C CNN
@@
 $EndComp
 $Comp
-L BreadBoardStrip BB8
+L BreadBoardStrip OUT3
 U 1 1 5A32E1BF
 P 5750 900
-F 0 "BB8" H 5909 937 60  0000 L CNN
+F 0 "OUT3" H 5909 937 60  0000 L CNN
 F 1 "BreadBoardStrip" H 5909 871 10  0000 L CNN
 F 2 "zfoot:BreadBoardStrip" H 5620 880 60  0001 C CNN
@@
 $EndComp
 $Comp
-L BreadBoardStrip BB11
+L BreadBoardStrip OUT2
 U 1 1 5A32E1FA
 P 4750 900
-F 0 "BB11" H 4909 937 60  0000 L CNN
+F 0 "OUT2" H 4909 937 60  0000 L CNN
 F 1 "BreadBoardStrip" H 4909 871 10  0000 L CNN
 F 2 "zfoot:BreadBoardStrip" H 4620 880 60  0001 C CNN
@@
 $EndComp
 $Comp
-L BreadBoardStrip BB12
-U 1 1 5A32E2E4
-P 6750 900
-F 0 "BB12" H 6909 937 60  0000 L CNN
-F 1 "BreadBoardStrip" H 6909 871 10  0000 L CNN
-F 2 "zfoot:BreadBoardStrip" H 6620 880 60  0001 C CNN
-F 3 "" H 6750 900 60  0001 C CNN
-	1    6750 900
-	1    0    0    -1
-$EndComp
-$Comp
-L BreadBoardStrip BB9
+L BreadBoardStrip IN2
 U 1 1 5A32E61E
 P 4300 900
-F 0 "BB9" H 4359 779 60  0000 C CNN
+F 0 "IN2" H 4359 779 60  0000 C CNN
 F 1 "BreadBoardStrip" H 4359 845 10  0000 C CNN
 F 2 "zfoot:BreadBoardStrip" H 4170 880 60  0001 C CNN
@@
 $EndComp
 $Comp
-L BreadBoardStrip BB10
-U 1 1 5A32E668
-P 6300 900
-F 0 "BB10" H 6359 779 60  0000 C CNN
-F 1 "BreadBoardStrip" H 6359 845 10  0000 C CNN
-F 2 "zfoot:BreadBoardStrip" H 6170 880 60  0001 C CNN
-F 3 "" H 6300 900 60  0001 C CNN
-	1    6300 900
-	-1   0    0    1
-$EndComp
-$Comp
-L BreadBoardStrip BB6
+L BreadBoardStrip IN3
 U 1 1 5A32E6B1
 P 5300 900
-F 0 "BB6" H 5359 779 60  0000 C CNN
+F 0 "IN3" H 5359 779 60  0000 C CNN
 F 1 "BreadBoardStrip" H 5359 845 10  0000 C CNN
 F 2 "zfoot:BreadBoardStrip" H 5170 880 60  0001 C CNN
@@
 F 3 "" H 4900 2600 60  0001 C CNN
 	7    4950 1950
-	1    0    0    -1
-$EndComp
-$Comp
-L GNDStrip PWR1
-U 1 1 5A330F13
-P 5000 1650
-F 0 "PWR1" H 5159 1687 15  0000 L CNN
-F 1 "PWRStrip" H 5159 1656 10  0000 L CNN
-F 2 "zfoot:GNDStrip" H 4870 1630 60  0001 C CNN
-F 3 "" H 5000 1650 60  0001 C CNN
-	1    5000 1650
 	1    0    0    -1
 $EndComp
@@
 	7200 2800 7250 2800
 $Comp
-L BreadBoardStrip BB1
+L BreadBoardStrip OscSwitchStrip1
 U 1 1 5A33DD61
 P 5550 1850
-F 0 "BB1" H 5609 1729 60  0000 C CNN
+F 0 "OscSwitchStrip1" H 5609 1729 60  0000 C CNN
 F 1 "BreadBoardStrip" H 5609 1795 10  0000 C CNN
 F 2 "zfoot:BreadBoardStrip" H 5420 1830 60  0001 C CNN
@@
 	-1   0    0    1
 $EndComp
+$Comp
+L GNDStrip PWR1
+U 1 1 5A330F13
+P 5000 1650
+F 0 "PWR1" H 5159 1687 15  0000 L CNN
+F 1 "PWRStrip" H 5159 1656 10  0000 L CNN
+F 2 "zfoot:GNDStrip" H 4870 1630 60  0001 C CNN
+F 3 "" H 5000 1650 60  0001 C CNN
+	1    5000 1650
+	1    0    0    -1
+$EndComp
+NoConn ~ 6300 900
+NoConn ~ 6750 900
 $EndSCHEMATC

Commit message: ready to send in
Parts:
- added GND2: GNDStrip, zfoot:GNDStripLONG, symbol GNDStrip
Connections:
- net at GND1.1, U2.7: now also GND2.1
Changed lines of the file:
@@
 NoConn ~ 6300 900
 NoConn ~ 6750 900
+$Comp
+L GNDStrip GND2
+U 1 1 5A336833
+P 5000 2250
+F 0 "GND2" H 5159 2287 15  0000 L CNN
+F 1 "GNDStrip" H 5159 2256 10  0000 L CNN
+F 2 "zfoot:GNDStripLONG" H 4870 2230 60  0001 C CNN
+F 3 "" H 5000 2250 60  0001 C CNN
+	1    5000 2250
+	0    1    1    0
+$EndComp
 $EndSCHEMATC
