File: workshop_drum2/workshop_drum2.sch (KiCad schematic (older format))
At the start: 28 parts, among them J1 9v_Battery_Clip, J2 Trigger_Input, J3 Output, U1 LM358, U2 7414, U3 78L05

Commit message: P1.1 - Updated footprints prior to deleting PCB
Parts:
- added C6: 10uF, 4ms-footprints:Cap_Electrolytic_TH, symbol 4ms-passives:CAP-ELEC-TH
- added DECAY_RANGE1: SPDT_small, zfoot:Switch_Toggle_SPDT_Mini_SolderLug, symbol zMECH:SPDT_small
- J2, J3: footprint zfoot:Jack_Instrument -> zfoot:Jack_Instrument_Bigger
- renumbered Switch_On1 to Button1
Connections:
- wire segments 62 -> 63
Other:
- moved on the sheet: C2
Changed lines of the file:
@@
 $EndComp
 $Comp
-L zMECH:SPST_small Switch_On1
+L zMECH:SPST_small Button1
 U 1 1 5A33654C
 P 1100 1200
-F 0 "Switch_On1" H 1100 1150 60  0000 C CNN
+F 0 "Button1" H 1100 1150 60  0000 C CNN
 F 1 "SPST_small" H 1100 1100 20  0000 C CNN
 F 2 "zfoot:SPST_Wired" H 1100 1200 60  0001 C CNN
@@
 F 0 "J2" H 650 1600 60  0000 C CNN
 F 1 "Trigger_Input" H 1100 1450 60  0000 C CNN
-F 2 "zfoot:Jack_Instrument" H 900 1500 60  0001 C CNN
+F 2 "zfoot:Jack_Instrument_Bigger" H 900 1500 60  0001 C CNN
 F 3 "" H 900 1500 60  0000 C CNN
 	1    900  1500
@@
 L 4ms-passives:CAP-ELEC-TH C2
 U 1 1 5A33B44F
-P 3250 1800
-F 0 "C2" H 3378 1792 45  0000 L CNN
-F 1 "1uF" H 3378 1708 45  0000 L CNN
-F 2 "4ms-footprints:Cap_Electrolytic_TH" H 3280 1950 20  0001 C CNN
-F 3 "" H 3250 1800 60  0001 C CNN
-	1    3250 1800
+P 3000 2100
+F 0 "C2" H 2850 2200 45  0000 L CNN
+F 1 "1uF" H 2850 2300 45  0000 L CNN
+F 2 "4ms-footprints:Cap_Electrolytic_TH" H 3030 2250 20  0001 C CNN
+F 3 "" H 3000 2100 60  0001 C CNN
+	1    3000 2100
 	1    0    0    -1
 $EndComp
@@
 L power1:GND #PWR013
 U 1 1 5A33BAE2
-P 3250 2000
-F 0 "#PWR013" H 3250 1750 50  0001 C CNN
-F 1 "GND" H 3255 1827 50  0000 C CNN
-F 2 "" H 3250 2000 50  0001 C CNN
-F 3 "" H 3250 2000 50  0001 C CNN
-	1    3250 2000
+P 3000 2300
+F 0 "#PWR013" H 3000 2050 50  0001 C CNN
+F 1 "GND" H 3005 2127 50  0000 C CNN
+F 2 "" H 3000 2300 50  0001 C CNN
+F 3 "" H 3000 2300 50  0001 C CNN
+	1    3000 2300
 	1    0    0    -1
 $EndComp
@@
 F 0 "J3" H 6450 2200 60  0000 C CNN
 F 1 "Output" H 6900 2050 60  0000 C CNN
-F 2 "zfoot:Jack_Instrument" H 6700 2100 60  0001 C CNN
+F 2 "zfoot:Jack_Instrument_Bigger" H 6700 2100 60  0001 C CNN
 F 3 "" H 6700 2100 60  0000 C CNN
 	1    6700 2100
@@
 Wire Wire Line
 	750  1200 950  1200
+$Comp
+L 4ms-passives:CAP-ELEC-TH C6
+U 1 1 5ABA2B19
+P 3300 2100
+F 0 "C6" H 3428 2092 45  0000 L CNN
+F 1 "10uF" H 3400 2200 45  0000 L CNN
+F 2 "4ms-footprints:Cap_Electrolytic_TH" H 3330 2250 20  0001 C CNN
+F 3 "" H 3300 2100 60  0001 C CNN
+	1    3300 2100
+	1    0    0    -1
+$EndComp
+$Comp
+L power1:GND #PWR0102
+U 1 1 5ABA2B77
+P 3300 2300
+F 0 "#PWR0102" H 3300 2050 50  0001 C CNN
+F 1 "GND" H 3305 2127 50  0000 C CNN
+F 2 "" H 3300 2300 50  0001 C CNN
+F 3 "" H 3300 2300 50  0001 C CNN
+	1    3300 2300
+	1    0    0    -1
+$EndComp
+$Comp
+L zMECH:SPDT_small DECAY_RANGE1
+U 1 1 5ABA4C11
+P 3250 1850
+F 0 "DECAY_RANGE1" V 3200 1550 60  0000 L CNN
+F 1 "SPDT_small" V 3303 1988 20  0000 L CNN
+F 2 "zfoot:Switch_Toggle_SPDT_Mini_SolderLug" H 3250 1850 60  0001 C CNN
+F 3 "" H 3250 1850 60  0001 C CNN
+	1    3250 1850
+	0    1    1    0
+$EndComp
+Wire Wire Line
+	3000 2000 3200 2000
 $EndSCHEMATC
