File: workshop_drum1.1/workshop_drum1.1.kicad_pcb (KiCad board)
At the start: 2 copper layers, 50 x 115 mm, 33 parts, among them J1 9v_Battery_Clip, J2 Trigger_Input, J3 Output, U1 LM358, U2 7414, U3 78L05

Commit message: Continued work on the pcb layout
Parts:
- moved R5 0.39 mm to (40.0, -89.7)
- moved R6 0.39 mm to (40.0, -85.3)
- moved R1 0.13 mm to (40.0, -99.1)
- moved R10 0.13 mm to (40.0, -76.2)
- moved R11 0.13 mm to (40.0, -80.5)
- moved R2 0.13 mm to (40.0, -67.1)
- moved R4 0.13 mm to (40.0, -71.6)
- moved R7 0.13 mm to (40.0, -103.6)
- moved R9 0.13 mm to (40.0, -94.5)
Routing:
- net GND: track 53.7 -> 226.7 mm, vias 0 -> 7
- net +5V: track 0.00 -> 83.3 mm, vias 0 -> 4
- net Net-(R1-Pad1): track 4.57 -> 80.7 mm, vias 0 -> 2
- net Net-(C2-Pad1): track 0.00 -> 63.7 mm, vias 0 -> 4
- net Net-(C4-Pad1): track 14.3 -> 68.8 mm, vias 0 -> 1
- net Net-(J2-Pad1): track 0.00 -> 46.2 mm, vias 0 -> 2
- net Net-(DECAY1-Pad2): track 45.3 -> 2.54 mm, vias 1 -> 0
- net Net-(C1-Pad1): track 0.00 -> 36.2 mm, vias 0 -> 2
- net Net-(R2-Pad1): track 0.00 -> 33.3 mm, vias 0 -> 2
- net Net-(SENSE/STARVE1-Pad2): track 0.00 -> 27.2 mm, vias 0 -> 2
- net Net-(R1-Pad2): track 0.00 -> 23.3 mm, vias 0 -> 3
- net Net-(U1-Pad1): track 0.00 -> 20.8 mm, vias 0 -> 2
- net Net-(D2-Pad2): track 0.00 -> 19.2 mm, vias 0 -> 2
- net Net-(J1-Pad1): track 0.00 -> 13.0 mm, vias 0 -> 1
- net Net-(D1-Pad2): track 0.00 -> 10.4 mm
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
Commit message: Ready for review
Parts:
- removed Switch_On1: SPST_small, zfoot:Jack_Instrument_Bigger
- added Button1: SPST_small, zfoot:Jack_Instrument_Bigger, F.Cu at (25.0, -111.0)
Routing:
- net GND: track 226.7 -> 300.6 mm, vias 7 -> 10
- net Net-(R10-Pad1): track 4.32 -> 66.8 mm, vias 0 -> 1
- net Net-(D1-Pad2): track 10.4 -> 66.6 mm, vias 0 -> 3
- net Net-(C2-Pad1): track 63.7 -> 109.5 mm, vias 4 -> 5
- net Net-(Osc_Select1-Pad1): track 0.00 -> 44.9 mm
- net Net-(DECAY1-Pad2): track 2.54 -> 45.8 mm
- net Net-(PITCH1-Pad1): track 2.54 -> 41.3 mm, vias 0 -> 1
- net Net-(D2-Pad2): track 19.2 -> 45.4 mm, vias 2 -> 3
- net Net-(PITCH1-Pad3): track 0.00 -> 21.6 mm, vias 0 -> 2
- net Net-(Osc_Select1-Pad3): track 12.7 -> 31.8 mm
- net Net-(Trig_LED1-Pad2): track 0.00 -> 12.8 mm
- net Net-(R8-Pad2): track 0.00 -> 10.6 mm
- net Net-(ON/OFF_LED1-Pad1): track 0.00 -> 8.28 mm
- net Net-(Button1-Pad1): track 23.3 -> 20.2 mm, vias 3 -> 2
- net +5V: track 83.3 -> 81.0 mm, vias 4 -> 3
