File: workshop_drum1.2/workshop_drum1.2.sch (KiCad schematic (older format))
At the start: 33 parts, among them J1 9v_Battery_Clip, J2 Trigger_Input, J3 Output, U1 LM358, U2 7414, U3 78L05

Commit message: -WIP-
Parts:
- removed R10: 470 after pot on output, 4ms-footprints:Resistor_TH_300, symbol 4ms-passives:RTH
- C2: value 1uF or smaller? -> 1uF
- DECAY1: value A100k-A1M -> A1M
- PITCH1: value B50k- try with A100k -> B50k
- R3: value 1k smaller is brighter -> 10k
- R4: value SET THIS TO ADJUST SENSE -> 100k
- R5: value 100k before decay pot -> 1k
- R6: value 470 before pot on non-inv input -> 1k
- R8: value 470 smaller is brighter -> 1k
- R9: value 1k - trig input resistor -> 1k
- SENSITIVITY1: renamed from SENSE/STARVE1; value A100k or bigger -> B100k
Connections:
- net at R11.2, U2.10: now also PITCH1.3 (Right)
Changed lines of the file:
@@
 EESchema Schematic File Version 4
-LIBS:workshop_drum1.1-cache
+LIBS:workshop_drum1.2-cache
 EELAYER 26 0
 EELAYER END
@@
 P 2400 3900
 F 0 "R3" V 2358 3968 45  0000 L CNN
-F 1 "1k smaller is brighter" V 2442 3968 45  0000 L CNN
+F 1 "10k" V 2442 3968 45  0000 L CNN
 F 2 "4ms-footprints:Resistor_TH_300" H 2430 4050 20  0001 C CNN
 F 3 "" H 2400 3900 60  0001 C CNN
@@
 $EndComp
 $Comp
-L 4ms-mech:POT SENSE/STARVE1
+L 4ms-mech:POT SENSITIVITY1
 U 1 1 5A337D75
 P 1800 1550
-F 0 "SENSE/STARVE1" H 1730 1596 50  0000 R CNN
-F 1 "A100k or bigger" H 1730 1505 50  0000 R CNN
+F 0 "SENSITIVITY1" H 1730 1596 50  0000 R CNN
+F 1 "B100k" H 1730 1505 50  0000 R CNN
 F 2 "zfoot:POT-9MM-ALPHA" H 2000 1300 50  0001 C CNN
 F 3 "" H 1800 1550 50  0001 C CNN
@@
 P 2500 2250
 F 0 "R4" H 2500 2150 45  0000 C CNN
-F 1 "SET THIS TO ADJUST SENSE" H 2450 2400 45  0000 C CNN
+F 1 "100k" H 2450 2400 45  0000 C CNN
 F 2 "4ms-footprints:Resistor_TH_300" H 2530 2400 20  0001 C CNN
 F 3 "" H 2500 2250 60  0001 C CNN
@@
 P 3250 1800
 F 0 "C2" H 3378 1792 45  0000 L CNN
-F 1 "1uF or smaller?" H 3378 1708 45  0000 L CNN
+F 1 "1uF" H 3378 1708 45  0000 L CNN
 F 2 "4ms-footprints:Cap_Electrolytic_TH" H 3280 1950 20  0001 C CNN
 F 3 "" H 3250 1800 60  0001 C CNN
@@
 P 3600 1900
 F 0 "R5" V 3650 1800 45  0000 C CNN
-F 1 "100k before decay pot" V 3550 1750 45  0000 C CNN
+F 1 "1k" V 3550 1750 45  0000 C CNN
 F 2 "4ms-footprints:Resistor_TH_300" H 3630 2050 20  0001 C CNN
 F 3 "" H 3600 1900 60  0001 C CNN
@@
 P 3600 2350
 F 0 "DECAY1" H 3530 2304 50  0000 R CNN
-F 1 "A100k-A1M" H 3530 2395 50  0000 R CNN
+F 1 "A1M" H 3530 2395 50  0000 R CNN
 F 2 "zfoot:POT-9MM-ALPHA" H 3800 2100 50  0001 C CNN
 F 3 "" H 3600 2350 50  0001 C CNN
@@
 P 4900 2500
 F 0 "R6" H 4950 2400 45  0000 C CNN
-F 1 "470 before pot on non-inv input" V 4950 1750 45  0000 C CNN
+F 1 "1k" H 4950 2300 45  0000 C CNN
 F 2 "4ms-footprints:Resistor_TH_300" H 4930 2650 20  0001 C CNN
 F 3 "" H 4900 2500 60  0001 C CNN
@@
 P 5350 2500
 F 0 "PITCH1" V 5236 2500 50  0000 C CNN
-F 1 "B50k- try with A100k" V 5145 2500 50  0000 C CNN
+F 1 "B50k" V 5145 2500 50  0000 C CNN
 F 2 "zfoot:POT-9MM-ALPHA" H 5550 2250 50  0001 C CNN
 F 3 "" H 5350 2500 50  0001 C CNN
@@
 P 7000 2800
 F 0 "R8" V 6958 2868 45  0000 L CNN
-F 1 "470 smaller is brighter" H 6950 3050 45  0000 L CNN
+F 1 "1k" H 6950 3050 45  0000 L CNN
 F 2 "4ms-footprints:Resistor_TH_300" H 7030 2950 20  0001 C CNN
 F 3 "" H 7000 2800 60  0001 C CNN
@@
 P 1550 1350
 F 0 "R9" H 1550 1156 45  0000 C CNN
-F 1 "1k - trig input resistor" H 1550 1240 45  0000 C CNN
+F 1 "1k" H 1550 1240 45  0000 C CNN
 F 2 "4ms-footprints:Resistor_TH_300" H 1580 1500 20  0001 C CNN
 F 3 "" H 1550 1350 60  0001 C CNN
@@
 Wire Wire Line
 	1800 1350 1800 1400
-$Comp
-L 4ms-passives:RTH R10
-U 1 1 5ABD3C3E
-P 5500 2250
-F 0 "R10" H 5550 2150 45  0000 C CNN
-F 1 "470 after pot on output" H 5800 2350 45  0000 C CNN
-F 2 "4ms-footprints:Resistor_TH_300" H 5530 2400 20  0001 C CNN
-F 3 "" H 5500 2250 60  0001 C CNN
-	1    5500 2250
-	0    1    1    0
-$EndComp
-Wire Wire Line
-	5500 2450 5500 2500
 Wire Wire Line
 	4500 1650 4950 1650
@@
 P 5750 1950
 F 0 "R11" H 5800 1850 45  0000 C CNN
-F 1 "1k" H 6050 2050 45  0000 C CNN
+F 1 "1k" H 5800 2100 45  0000 C CNN
 F 2 "4ms-footprints:Resistor_TH_300" H 5780 2100 20  0001 C CNN
 F 3 "" H 5750 1950 60  0001 C CNN
@@
 Wire Wire Line
 	5550 1950 5500 1950
-Wire Wire Line
-	5500 2050 5500 1950
 Connection ~ 5500 1950
 Wire Wire Line
@@
 Wire Wire Line
 	700  1150 700  1050
+Wire Wire Line
+	5500 1950 5500 2500
 $EndSCHEMATC

Commit message: About to update from SCHEM after doing logos
Parts:
- added LOGO1: Open, zfoot:Logo_Open-1, symbol 4ms-passives:C
- added LOGO2: S1, zfoot:Logo_S1-2, symbol 4ms-passives:C
- added LOGO3: OSH, zfoot:Logo_OSH-1, symbol 4ms-passives:C
- BreadBoardStrip1: renamed from PathToSwitch1; value BreadBoardStrip -> Path to Switch
- C5: value 100nf-220nF or bigger? -> 100nf
- J1: value 9v_Battery_Clip -> 9v; footprint zfoot:Jack_Instrument_Bigger -> zfoot:9v_Bigger
- J2: value Trigger_Input -> INPUT
- J3: value Output -> OUTPUT
- LED1: renamed from ON/OFF_LED1; value LED-C1-A2 -> ON!
- LED2: renamed from Trig_LED1; value LED-C1-A2 -> SIGNAL
- SW1: renamed from PWR2; value SPST_small -> POWER
- SW2: renamed from Osc_Select1; value SPDT_small -> OSCILLATOR SELECT
- SW3: renamed from Button1; value SPST_small -> BUTTON; footprint zfoot:Jack_Instrument_Bigger -> zfoot:Button_Bigger
Changed lines of the file:
@@
 P 1100 3400
 F 0 "J1" H 1131 3837 60  0000 C CNN
-F 1 "9v_Battery_Clip" H 1131 3731 60  0000 C CNN
-F 2 "zfoot:Jack_Instrument_Bigger" H 1100 3400 60  0001 C CNN
+F 1 "9v" H 1131 3731 60  0000 C CNN
+F 2 "zfoot:9v_Bigger" H 1100 3400 60  0001 C CNN
 F 3 "" H 1100 3400 60  0001 C CNN
 	1    1100 3400
@@
 $EndComp
 $Comp
-L 4ms-passives:LED-C1-A2 ON/OFF_LED1
+L 4ms-passives:LED-C1-A2 LED1
 U 1 1 5A333512
 P 2250 3700
-F 0 "ON/OFF_LED1" H 2300 3496 45  0000 C CNN
-F 1 "LED-C1-A2" H 2300 3580 45  0000 C CNN
+F 0 "LED1" H 2300 3496 45  0000 C CNN
+F 1 "ON!" H 2300 3580 45  0000 C CNN
 F 2 "zfoot:LED_D5.0mm" H 2280 3850 20  0001 C CNN
 F 3 "" H 2250 3700 60  0001 C CNN
@@
 P 6400 1900
 F 0 "C5" V 6350 1950 50  0000 L CNN
-F 1 "100nf-220nF or bigger?" V 6550 1800 50  0000 L CNN
+F 1 "100nf" V 6550 1800 50  0000 L CNN
 F 2 "4ms-footprints:Cap_Ceramic_TH" H 6438 1750 50  0001 C CNN
 F 3 "" H 6400 1900 50  0001 C CNN
@@
 $EndComp
 $Comp
-L zMECH:SPDT_small Osc_Select1
+L zMECH:SPDT_small SW2
 U 1 1 5A3358B6
 P 6100 1900
-F 0 "Osc_Select1" H 6000 1750 60  0000 C CNN
-F 1 "SPDT_small" H 6100 2060 20  0000 C CNN
+F 0 "SW2" H 6000 1750 60  0000 C CNN
+F 1 "OSCILLATOR SELECT" H 6100 2060 20  0000 C CNN
 F 2 "zfoot:Switch_Toggle_SPDT_Mini_SolderLug" H 6100 1900 60  0001 C CNN
 F 3 "" H 6100 1900 60  0001 C CNN
@@
 $EndComp
 $Comp
-L zMECH:SPST_small PWR2
+L zMECH:SPST_small SW1
 U 1 1 5A335D0A
 P 1800 3250
-F 0 "PWR2" H 1800 3484 60  0000 C CNN
-F 1 "SPST_small" H 1800 3410 20  0000 C CNN
+F 0 "SW1" H 1800 3484 60  0000 C CNN
+F 1 "POWER" H 1800 3410 20  0000 C CNN
 F 2 "zfoot:Switch_Toggle_SPST_Mini_SolderLug_2legs" H 1800 3250 60  0001 C CNN
 F 3 "" H 1800 3250 60  0001 C CNN
@@
 $EndComp
 $Comp
-L zMECH:SPST_small Button1
+L zMECH:SPST_small SW3
 U 1 1 5A33654C
 P 1150 1150
-F 0 "Button1" H 1150 1100 60  0000 C CNN
-F 1 "SPST_small" H 1150 1050 20  0000 C CNN
-F 2 "zfoot:Jack_Instrument_Bigger" H 1150 1150 60  0001 C CNN
+F 0 "SW3" H 1150 1100 60  0000 C CNN
+F 1 "BUTTON" H 1150 1050 20  0000 C CNN
+F 2 "zfoot:Button_Bigger" H 1150 1150 60  0001 C CNN
 F 3 "" H 1150 1150 60  0001 C CNN
 	1    1150 1150
@@
 P 900 1500
 F 0 "J2" H 650 1600 60  0000 C CNN
-F 1 "Trigger_Input" H 1100 1450 60  0000 C CNN
+F 1 "INPUT" H 1100 1450 79  0000 C CNN
 F 2 "zfoot:Jack_Instrument_Bigger" H 900 1500 60  0001 C CNN
 F 3 "" H 900 1500 60  0000 C CNN
@@
 P 7450 2050
 F 0 "J3" H 7200 2150 60  0000 C CNN
-F 1 "Output" H 7650 2000 60  0000 C CNN
+F 1 "OUTPUT" H 7650 2000 60  0000 C CNN
 F 2 "zfoot:Jack_Instrument_Bigger" H 7450 2050 60  0001 C CNN
 F 3 "" H 7450 2050 60  0000 C CNN
@@
 	5850 2800 5850 2850
 $Comp
-L 4ms-passives:LED-C1-A2 Trig_LED1
+L 4ms-passives:LED-C1-A2 LED2
 U 1 1 5A332943
 P 6600 2800
-F 0 "Trig_LED1" H 6650 2596 45  0000 C CNN
-F 1 "LED-C1-A2" H 6650 2680 45  0000 C CNN
+F 0 "LED2" H 6650 2596 45  0000 C CNN
+F 1 "SIGNAL" H 6650 2680 45  0000 C CNN
 F 2 "zfoot:LED_D5.0mm" H 6630 2950 20  0001 C CNN
 F 3 "" H 6600 2800 60  0001 C CNN
@@
 	7200 2800 7250 2800
 $Comp
-L zMECH:BreadBoardStrip PathToSwitch1
+L zMECH:BreadBoardStrip BreadBoardStrip1
 U 1 1 5A33DD61
 P 5950 1850
-F 0 "PathToSwitch1" H 6000 2000 60  0000 C CNN
-F 1 "BreadBoardStrip" H 6009 1795 10  0000 C CNN
+F 0 "BreadBoardStrip1" H 6000 2000 60  0000 C CNN
+F 1 "Path to Switch" H 6009 1795 10  0000 C CNN
 F 2 "zfoot:BREAKOUTswitch" H 5820 1830 60  0001 C CNN
 F 3 "" H 5950 1850 60  0001 C CNN
@@
 Wire Wire Line
 	5500 1950 5500 2500
+$Comp
+L 4ms-passives:C LOGO1
+U 1 1 5ADBC7A3
+P 5800 4050
+F 0 "LOGO1" H 5915 4096 50  0000 L CNN
+F 1 "Open" H 5915 4005 50  0000 L CNN
+F 2 "zfoot:Logo_Open-1" H 5838 3900 50  0001 C CNN
+F 3 "" H 5800 4050 50  0001 C CNN
+	1    5800 4050
+	1    0    0    -1
+$EndComp
+$Comp
+L 4ms-passives:C LOGO2
+U 1 1 5ADBC845
+P 6150 4000
+F 0 "LOGO2" H 6265 4046 50  0000 L CNN
+F 1 "S1" H 6265 3955 50  0000 L CNN
+F 2 "zfoot:Logo_S1-2" H 6188 3850 50  0001 C CNN
+F 3 "" H 6150 4000 50  0001 C CNN
+	1    6150 4000
+	1    0    0    -1
+$EndComp
+$Comp
+L 4ms-passives:C LOGO3
+U 1 1 5ADBC8AF
+P 6600 4050
+F 0 "LOGO3" H 6715 4096 50  0000 L CNN
+F 1 "OSH" H 6715 4005 50  0000 L CNN
+F 2 "zfoot:Logo_OSH-1" H 6638 3900 50  0001 C CNN
+F 3 "" H 6600 4050 50  0001 C CNN
+	1    6600 4050
+	1    0    0    -1
+$EndComp
 $EndSCHEMATC
