File: workshop_drum1.2/workshop_drum1.2.kicad_pcb (KiCad board)
At the start: 2 copper layers, 50 x 115 mm, 33 parts, among them J1 9v_Battery_Clip, J2 Trigger_Input, J3 Output, U1 LM358, U2 7414, U3 78L05

Commit message: -WIP-
Parts:
- removed R10: 470 after pot on output, 4ms-footprints:Resistor_TH_300
- C2: value 1uF or smaller? -> 1uF
- DECAY1: value A100k-A1M -> A1M
- PITCH1: value B50k- try with A100k -> B50k
- R3: value 1k smaller is brighter -> 10k
- R4: value SET THIS TO ADJUST SENSE -> 100k
- R5: value 100k before decay pot -> 1k
- R6: value 470 before pot on non-inv input -> 1k
- R8: value 470 smaller is brighter -> 1k
- R9: value 1k - trig input resistor -> 1k
- SENSITIVITY1: renamed from SENSE/STARVE1; value A100k or bigger -> B100k
- moved PITCH1 44.0 mm to (104.1, 88.9)
- moved SENSITIVITY1 35.4 mm to (99.8, 110.0)
Connections:
- R11 pad 2: Net-(R10-Pad1) -> Net-(PITCH1-Pad3)
- U2 pad 10: Net-(R10-Pad1) -> Net-(PITCH1-Pad3)
Routing:
- net Net-(R10-Pad1): track 66.8 -> 0.00 mm, vias 1 -> 0
- net Net-(PITCH1-Pad3): track 21.6 -> 88.4 mm, vias 2 -> 3

Commit message: About to update from SCHEM after doing logos
Parts:
- removed Button1: SPST_small, zfoot:Jack_Instrument_Bigger
- added LOGO1: Open, zfoot:Logo_Open-1, B.Cu at (134.9, 69.6)
- added LOGO3: OSH, zfoot:Logo_OSH-1, B.Cu at (148.1, 48.8)
- added S1: LOGO2, zfoot:Logo_S1-2, B.Cu at (159.0, 72.4)
- added SW3: BUTTON, zfoot:Button_Bigger, F.Cu at (147.9, 41.4)
- BreadBoardStrip1: renamed from PathToSwitch1; value BreadBoardStrip -> Path to Switch
- C5: value 100nf-220nF or bigger? -> 100nf
- J1: value 9v_Battery_Clip -> 9v; footprint zfoot:Jack_Instrument_Bigger -> zfoot:9v_Bigger
- J2: value Trigger_Input -> INPUT
- J3: value Output -> OUTPUT
- LED1: renamed from ON/OFF_LED1; value LED-C1-A2 -> ON!
- LED2: renamed from Trig_LED1; value LED-C1-A2 -> SIGNAL
- SW1: renamed from PWR2; value SPST_small -> POWER
- SW2: renamed from Osc_Select1; value SPDT_small -> OSCILLATOR SELECT
- moved SENSITIVITY1 55.5 mm to (147.6, 81.8)
- moved PITCH1 30.0 mm to (132.9, 97.4)
- moved R2 9.09 mm to (162.9, 76.2)
Routing:
- net Net-(R1-Pad1): track 80.7 -> 50.1 mm, vias 2 -> 1
- net Net-(PITCH1-Pad1): track 41.3 -> 71.8 mm, vias 1 -> 2
- net Net-(SENSITIVITY1-Pad2): track 27.2 -> 10.2 mm, vias 2 -> 1
- net GND: track 300.6 -> 297.4 mm
- net Net-(R2-Pad1): track 33.3 -> 36.1 mm
- net Net-(PITCH1-Pad3): track 88.4 -> 89.9 mm, vias 3 -> 2
- net Net-(D2-Pad2): track 45.4 -> 44.3 mm

Commit message: Made PCB look cool - but havent updated from sch yet
Parts:
- removed LOGO1: Open, zfoot:Logo_Open-1
- removed S1: LOGO2, zfoot:Logo_S1-2
- added G***: LOGO, zfoot:Logo_MD-P3-2, B.Cu at (215.4, 59.7)
- added G***: LOGO, zfoot:Logo_MD-Battery, B.Cu at (203.7, 114.3)
- added G***: LOGO, zfoot:Logo_MNT-2, B.Cu at (147.8, 126.0)
- added G***: LOGO, zfoot:Logo_Open-3, B.Cu at (130.8, 116.1)
- added LOGO2: S1, zfoot:Logo_S1-2, B.Cu at (159.3, 62.5)
- LOGO3: footprint zfoot:Logo_OSH-1 -> zfoot:Logo_OSH-3
- moved LOGO3 34.3 mm to (140.7, 82.3)
Other:
- board text added: "A DRUM SYNTH CIRCUIT BY"
- board text added: "DRUM"
- board text added: "MOSS"
- board text added: "P3"
- board text added: "ZACH D'AGOSTINO & NOA VER"
